Commit message: frist_commit

File: urdf/bodot.urdf (robot description, URDF)
Before this commit: robot low_level, 9 links, 8 joints
Links:
- removed link base_laser_link
- removed link caster_link_2
- removed link caster_link_3
- added link base_laser; visual cylinder length=0.04 radius=0.035
- link base_link: geometry visual box size=0.29 0.29 0.26
- link caster_link_1: geometry visual cylinder length=0.02 radius=0.04
- link imu_link: geometry 
- link wheel_left_link: geometry visual cylinder length=0.05 radius=0.04
- link wheel_right_link: geometry visual cylinder length=0.05 radius=0.04
Joints:
- removed joint base_laser
- removed joint caster_joint_2
- removed joint caster_joint_3
- added joint scan_joint: type fixed, parent base_link, child base_laser, origin xyz=0.105 0 0.15 rpy=0 0 -3.14
- joint base_joint: child base_footprint -> base_link; origin xyz=0.2 0.15 0 rpy=0 0 0 -> xyz=0.0 0.0 0.0 rpy=0 0 0; parent base_link -> base_footprint
- joint caster_joint_1: origin xyz=0.19 0 -0.1 rpy=-1.57 0 0 -> xyz=-0.145 0 -0.145 rpy=-1.57 0 0
- joint imu_joint: origin xyz=0.05 0 0.1015 rpy=0 0 0 -> xyz=0 0 0 rpy=0 0 1.57
- joint wheel_left_joint: axis (none) -> 0 0 1; origin xyz=0 0.2 -0.075 rpy=1.57 0 0 -> xyz=0.11 0.17 -0.145 rpy=-1.57 0 0
- joint wheel_right_joint: axis (none) -> 0 0 1; origin xyz=0 -0.2 -0.075 rpy=1.57 0 0 -> xyz=0.11 -0.17 -0.145 rpy=-1.57 0 0
